File: hardware/porcupine5v1_2.brd (EAGLE design)
At the start: 28.5 x 29.7 mm, 44 parts, among them X1 PROGCON

Commit message: updated oled board
Parts:
- moved U$2 45.3 mm to (7.34, 20.3), flipped to the bottom
- moved U$3 41.7 mm to (4.09, 15.2), flipped to the bottom, turned to 270 degrees
- moved U$1 38.0 mm to (5.84, 27.4), flipped to the bottom, turned to 90 degrees
- moved R5 31.7 mm to (3.20, 10.5), flipped to the bottom
- moved R3 29.1 mm to (3.20, 12.5), flipped to the bottom
- moved C_PWR_SW 4.88 mm to (1.50, 21.9), turned to 270 degrees
- moved C2_32KHZ 2.71 mm to (5.49, 22.1), turned to 180 degrees
- moved C1_32KHZ 2.27 mm to (8.79, 22.1)
- moved SDCARD_CON 0.46 mm to (14.5, 14.8)
- moved CHARGER 0.22 mm to (5.71, 27.1), turned to 270 degrees
- moved R4 0.08 mm to (10.7, 4.42)
Routing:
- net PWRGD: track 0.00 -> 38.1 mm, vias 0 -> 4
- net POK: track 0.00 -> 33.3 mm, vias 0 -> 5
- net GND: track 188.0 -> 210.5 mm
- net N$2: track 0.00 -> 5.11 mm
- net N$1: track 0.00 -> 4.04 mm
- net +3V3: track 178.7 -> 182.4 mm, vias 11 -> 12
- net N$6: track 7.21 -> 4.84 mm, vias 1 -> 0
- net SDO_SPI&D6_OLED@RD6: track 56.2 -> 58.3 mm
- net V_BAT: track 22.8 -> 20.9 mm, vias 1 -> 0
- net N$3: track 7.68 -> 6.77 mm, vias 1 -> 0
- net PROG_CLK@RB6: track 11.1 -> 11.8 mm
- net SDI: track 23.1 -> 22.4 mm
- net SCLK: track 69.7 -> 70.3 mm
- net PROG_DATA@RB7: track 12.6 -> 13.2 mm
- net VUSB: track 23.6 -> 23.1 mm, vias 2 -> 1
